File: MOS6551-ATMEGA8535/MOS6551-ATmega8535.sch (KiCad schematic (older format))
At the start: 8 parts, among them J1 Conn_02x03_Odd_Even, J2 Conn_02x14_Counter_Clockwise, U1 ATmega8535-16AU, Y1 Crystal

Commit message: Another darft
Parts:
- removed J2: Conn_02x14_Counter_Clockwise, Package_DIP:DIP-28_W15.24mm_Socket, symbol Connector_Generic:Conn_02x14_Counter_Clockwise
- removed U1: ATmega8535-16AU, Package_QFP:TQFP-44_10x10mm_P0.8mm, symbol MCU_Microchip_ATmega:ATmega8535-16AU
- added C10, C6, C8: 1nF, Capacitor_SMD:C_1206_3216Metric, symbol Device:C_Small
- added C5, C7, C9: 1µF, Capacitor_SMD:C_1206_3216Metric, symbol Device:C_Small
- added J2: Conn_02x02_Counter_Clockwise, Connector_PinHeader_2.54mm:PinHeader_2x02_P2.54mm_Vertical_SMD, symbol Connector_Generic:Conn_02x02_Counter_Clockwise
- added J3, J4: Conn_01x14, Connector_PinHeader_2.54mm:PinHeader_1x14_P2.54mm_Vertical_SMD_Pin1Left, symbol Connector_Generic:Conn_01x14
- added U1: ATmega88-20AU, Package_QFP:TQFP-32_7x7mm_P0.8mm, symbol MCU_Microchip_ATmega:ATmega88-20AU
- added U2: XC9572XL-VQ64, Package_QFP:TQFP-64_10x10mm_P0.5mm, symbol CPLD_Xilinx:XC9572XL-VQ64
- added U3: MCP1700-3302E_SOT23, Package_TO_SOT_SMD:SOT-23, symbol Regulator_Linear:MCP1700-3302E_SOT23
Connections:
- net labels added: +3.3V
- wire segments 92 -> 171
Other:
- moved on the sheet: C1, C2, C3, C4, J1, Y1
